File: NUS-MDM-10.kicad_pcb (KiCad board)
At the start: 2 copper layers, 102 x 79 mm, 80 parts, among them J1 Edge_Connector, K1 NEC EG2-3, Q1 2SC4081 BQ NPN, Q2 2SC3444-E DE NPN, T1 A202 9N III, U1 AE LDO, U3 RJ11_Shielded, Y1 D102K9

Commit message: Add files via upload
Connections:
- net /+IN1 renamed Net-(U4-+IN1)
- net /+IN2 renamed Net-(U4-+IN2)
- net /-IN1 renamed Net-(U4--IN1)
- net /-IN2 renamed Net-(U4--IN2)
- net /C19 renamed /NUS.P20
- net /C22.Neg renamed /NUS.P28
- net /LED.Neg renamed Net-(D3-K)
- net /LED.Pos renamed Net-(D3-A)
- net /OUT1 renamed Net-(U4-OUT1)
- net /OUT1.Sense renamed /NUS.P27-30-32
- net /OUT1.adj renamed /NUS.P31
- net /OUT2 renamed Net-(U4-OUT2)
- net /PC1.P2 renamed Net-(PC1-C,A)
- net /Q1.Base renamed Net-(Q1-B_(1))
- net /Q1.Collector renamed Net-(D2-A)
- net /Q2.Base renamed Net-(D6-K)
- net /Q2.Emitter renamed Net-(Q2-E_(3))
- net /RJ11.D5+ renamed Net-(D5-+)
- net /RJ11.D5- renamed Net-(D5--)
- net /RJ11.K1 renamed Net-(D5-Pad3)
- net /RJ11.P3 renamed Net-(PC1-A,C)
- net /RJ11.P4 renamed Net-(C14-Pad2)
- net /T1.P2 renamed Net-(D6-A)
- net /T1_Coil renamed Net-(T1-S2)
