File: NUS-MDM-10.kicad_sch (KiCad schematic)
At the start: 76 parts, among them J2 Edge_Connector, K1 NEC EG2-3, Q1 2SC4081 BQ NPN, Q2 2SC3444-E DE NPN, T1 A202 9N III, U1 AE LDO, U3 RJ11_Shielded, Y1 D102K9

Commit message: Add files via upload
Connections:
- net +IN1: no longer names the net of R11.1, R13.1, U4.3 (+IN1)
- net +IN2: no longer names the net of C20.2, R10.1, R6.2, U4.5 (+IN2)
- net -IN1: no longer names the net of R12.1, R18.1, U4.2 (-IN1)
- net -IN2: no longer names the net of C13.1, R4.1, R8.1, U4.6 (-IN2)
- net C19 renamed NUS.P20
- net C22.Neg renamed NUS.P28
- net LED.Neg: no longer names the net of D3.1 (K), K1.7
- net LED.Pos: no longer names the net of D3.2 (A), R5.2
- net OUT1: no longer names the net of C30.2, R18.2, R19.1, U4.1 (OUT1)
- net OUT1.Sense renamed NUS.P27-30-32
- net OUT1.adj renamed NUS.P31
- net OUT2: no longer names the net of C13.2, R11.2, R4.2, R7.2, R9.1, U4.7 (OUT2)
- net PC1.P2: no longer names the net of D1.1 (K), PC1.2 (C,A)
- net Q1.Base: no longer names the net of Q1.1 (B_(1)), R2.2
- net Q1.Collector: no longer names the net of D2.2 (A), K1.10, Q1.3 (C_(3))
- net Q2.Base: no longer names the net of C31.1, D6.1 (K), Q2.1 (B_(1)), R14.2, R15.1
- net Q2.Emitter: no longer names the net of Q2.3 (E_(3)), R15.2, R17.2
- net RJ11.D5+: no longer names the net of C18.1, D5.1 (+), Q2.2 (C_(2)), R14.1, RV2.2
- net RJ11.D5-: no longer names the net of C31.2, D5.2 (-), R17.1, RV2.1, T1.1 (PR1)
- net RJ11.K1: no longer names the net of D5.3, K1.4
- net RJ11.P3: no longer names the net of K1.3, PC1.1 (A,C), RV1.2, U3.3
- net RJ11.P4: no longer names the net of C14.2, D5.4, RV1.1, U3.4
- net T1.P2: no longer names the net of C18.2, D6.2 (A), T1.2 (PM)
- net T1_Coil: no longer names the net of C17.2, D4.1, T1.5 (S2)
Other:
- moved on the sheet: C1, C10, C11, C12, C13, C14, C15, C17, C18, C19, C2, C20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
